File: PCB/MusicDevice.kicad_sch (KiCad schematic)
At the start: 11 parts, among them J1 Capacitive Touch Buttons, SW1 SW_Push, SW2 SW_Push, SW3 SW_Push, SW4 RotaryEncoder_Switch_MP, U1 Waveshare ESP32-S3-ZERO

Commit message: Reorganized File structure, separating pcn and model
Changed lines of the file:
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@@
 		(at 161.29 31.75)
+	)
+	(bus_entry
+		(at -360.68 78.74)
+		(size 2.54 2.54)
+		(stroke
+			(width 0)
+			(type default)
+		)
+	)
+	(bus_entry
+		(at 49.53 86.36)
+		(size 2.54 2.54)
+		(stroke
+			(width 0)
+			(type default)
+		)
 	)
 	(wire
